Commit message: leap hand dummy urdf update

File: robots/hands/leap_hand/leap_hand_right_dummy_ball.urdf (robot description, URDF)
Before this commit: robot leap_right, 28 links, 27 joints
Links:
- removed link pip_4
- added link thumb_temp_base, mass 0.032; collision box size=0.034 0.026 0.022; visual mesh filename=meshes/visual/pip.obj
- link fingertip: geometry collision box size=0.014 0.022 0.004; collision box size=0.014 0.022 0.004
- link fingertip_2: geometry collision box size=0.014 0.022 0.004; collision box size=0.014 0.022 0.004
- link fingertip_3: geometry collision box size=0.014 0.022 0.004; collision box size=0.014 0.022 0.004
- link thumb_fingertip: geometry collision box size=0.008 0.024 0.018; collision box size=0.02 0.004 0.03
Joints:
- joint 12: child pip_4 -> thumb_temp_base
- joint 13: parent pip_4 -> thumb_temp_base
- joint base_joint: parent base_link_yaw -> base
- joint dummy_x_rotation_joint: child base_link_roll -> base_link_pitch; parent base_link_z -> base_link_roll
- joint dummy_x_translation_joint: child base_link_x -> base_link_y; parent base -> base_link_x
- joint dummy_y_rotation_joint: child base_link_pitch -> base_link_yaw; parent base_link_roll -> base_link_pitch
- joint dummy_y_translation_joint: child base_link_y -> base_link_z; parent base_link_x -> base_link_y
- joint dummy_z_rotation_joint: child base_link_yaw -> base; parent base_link_pitch -> base_link_yaw
- joint dummy_z_translation_joint: child base_link_z -> base_link_roll; parent base_link_y -> base_link_z
