Commit message: refine the barrett hand model, add barrett and allegro left pc

File: robots/hands/barrett_hand/bhand_model_dummy_ball_balls.urdf (robot description, URDF)
Before this commit: robot bhand_model, 56 links, 55 joints
Links:
- removed link base_link_collision_ball_10
- removed link base_link_collision_ball_11
- removed link base_link_collision_ball_12
- removed link base_link_collision_ball_7
- removed link base_link_collision_ball_8
- removed link base_link_collision_ball_9
- link base_link: geometry collision box size=0.026 0.02 0.01; collision box size=0.026 0.02 0.01
- link base_link_collision_ball_0: geometry collision sphere radius=0.02; visual sphere radius=0.02
- link base_link_collision_ball_1: geometry collision sphere radius=0.02; visual sphere radius=0.02
- link base_link_collision_ball_2: geometry collision sphere radius=0.02; visual sphere radius=0.02
- link base_link_collision_ball_3: geometry collision sphere radius=0.02; visual sphere radius=0.02
- link base_link_collision_ball_4: geometry collision sphere radius=0.05; visual sphere radius=0.05
- link base_link_collision_ball_5: geometry collision sphere radius=0.032; visual sphere radius=0.032
- link base_link_collision_ball_6: geometry collision sphere radius=0.032; visual sphere radius=0.032
Joints:
- removed joint base_link_collision_ball_10_joint
- removed joint base_link_collision_ball_11_joint
- removed joint base_link_collision_ball_12_joint
- removed joint base_link_collision_ball_7_joint
- removed joint base_link_collision_ball_8_joint
- removed joint base_link_collision_ball_9_joint
- joint base_link_collision_ball_0_joint: origin xyz=0.0 0.0 0.02  rpy=0 0 0 -> xyz=0.0 0.028 0.056  rpy=0 0 0
- joint base_link_collision_ball_1_joint: origin xyz=0.0 0.024  0.02  rpy=0 0 0 -> xyz=0.0 -0.028 0.056  rpy=0 0 0
- joint base_link_collision_ball_2_joint: origin xyz=0.0 0.024  0.02  rpy=0 0 0 -> xyz=0.0 -0.05 0.056  rpy=0 0 0
- joint base_link_collision_ball_3_joint: origin xyz=0.0 -0.024  0.02  rpy=0 0 0 -> xyz=0.0 -0.05 0.075  rpy=0 0 0
- joint base_link_collision_ball_4_joint: origin xyz=0.028 0.0  0.015  rpy=0 0 0 -> xyz=0.0 0.0 0.032  rpy=0 0 0
- joint base_link_collision_ball_5_joint: origin xyz=-0.02 0.02  0.016  rpy=0 0 0 -> xyz=0.022 0.0 0.051  rpy=0 0 0
- joint base_link_collision_ball_6_joint: origin xyz=-0.02 -0.02  0.016  rpy=0 0 0 -> xyz=-0.022 0.0 0.051  rpy=0 0 0
