Commit message: panda and shadow refine

File: robots/hands/panda_gripper/panda_gripper_dummy_ball_balls.urdf (robot description, URDF)
Before this commit: robot panda_gripper, 10 links, 10 joints
Links:
- added link base_link_x
- added link panda_hand_collision_ball_1; collision sphere radius=0.0460; visual sphere radius=0.0460
- added link panda_hand_collision_ball_2; collision sphere radius=0.0460; visual sphere radius=0.0460
- added link panda_leftfinger_collision_ball_0; collision sphere radius=0.0120; visual sphere radius=0.0120
- added link panda_leftfinger_collision_ball_1; collision sphere radius=0.0120; visual sphere radius=0.0120
- added link panda_leftfinger_collision_ball_2; collision sphere radius=0.0120; visual sphere radius=0.0120
- added link panda_rightfinger_collision_ball_0; collision sphere radius=0.0120; visual sphere radius=0.0120
- added link panda_rightfinger_collision_ball_1; collision sphere radius=0.0120; visual sphere radius=0.0120
- added link panda_rightfinger_collision_ball_2; collision sphere radius=0.0120; visual sphere radius=0.0120
- link panda_hand_collision_ball_0: geometry collision sphere radius=0.0460; visual sphere radius=0.0460
Joints:
- added joint panda_hand_collision_ball_1_joint: type fixed, parent panda_hand, child panda_hand_collision_ball_1, origin xyz=0.0 -0.06 0.024 rpy=0 0 0
- added joint panda_hand_collision_ball_2_joint: type fixed, parent panda_hand, child panda_hand_collision_ball_2, origin xyz=0.0 0.06 0.024 rpy=0 0 0
- added joint panda_leftfinger_collision_ball_0_joint: type fixed, parent panda_leftfinger, child panda_leftfinger_collision_ball_0, origin xyz=0.0 0.02 0.014 rpy=0 0 0
- added joint panda_leftfinger_collision_ball_1_joint: type fixed, parent panda_leftfinger, child panda_leftfinger_collision_ball_1, origin xyz=0.0 0.019 0.029 rpy=0 0 0
- added joint panda_leftfinger_collision_ball_2_joint: type fixed, parent panda_leftfinger, child panda_leftfinger_collision_ball_2, origin xyz=0.0 0.009 0.045 rpy=0 0 0
- added joint panda_rightfinger_collision_ball_0_joint: type fixed, parent panda_rightfinger, child panda_rightfinger_collision_ball_0, origin xyz=0.0 -0.02 0.014 rpy=0 0 0
- added joint panda_rightfinger_collision_ball_1_joint: type fixed, parent panda_rightfinger, child panda_rightfinger_collision_ball_1, origin xyz=0.0 -0.019 0.029 rpy=0 0 0
- added joint panda_rightfinger_collision_ball_2_joint: type fixed, parent panda_rightfinger, child panda_rightfinger_collision_ball_2, origin xyz=0.0 -0.009 0.045 rpy=0 0 0
- joint panda_hand_collision_ball_0_joint: origin xyz=0.0 0.0 0.02  rpy=0 0 0 -> xyz=0.0 0.0 0.024 rpy=0 0 0

File: robots/hands/shadow_hand/shadow_hand_right_dummy_ball_balls.urdf (robot description, URDF)
Before this commit: robot shadow_right, 83 links, 82 joints
Links:
- added link palm_collision_ball_10; collision sphere radius=0.013; visual sphere radius=0.013
- added link palm_collision_ball_11; collision sphere radius=0.013; visual sphere radius=0.013
- added link palm_collision_ball_4; collision sphere radius=0.013; visual sphere radius=0.013
- added link palm_collision_ball_5; collision sphere radius=0.013; visual sphere radius=0.013
- added link palm_collision_ball_6; collision sphere radius=0.013; visual sphere radius=0.013
- added link palm_collision_ball_7; collision sphere radius=0.013; visual sphere radius=0.013
- added link palm_collision_ball_8; collision sphere radius=0.013; visual sphere radius=0.013
- added link palm_collision_ball_9; collision sphere radius=0.013; visual sphere radius=0.013
- link palm: geometry collision box size=0.018 0.024 0.004; collision box size=0.020 0.024 0.032
Joints:
- added joint palm_collision_ball_10_joint: type fixed, parent palm, child palm_collision_ball_10, origin xyz=0.0 0.0 0.082 rpy=0 0 0
- added joint palm_collision_ball_11_joint: type fixed, parent palm, child palm_collision_ball_11, origin xyz=0.02 0.0 0.076 rpy=0 0 0
- added joint palm_collision_ball_4_joint: type fixed, parent palm, child palm_collision_ball_4, origin xyz=0.0 0.0 0.004  rpy=0 0 0
- added joint palm_collision_ball_5_joint: type fixed, parent palm, child palm_collision_ball_5, origin xyz=0.0 0.0 0.026  rpy=0 0 0
- added joint palm_collision_ball_6_joint: type fixed, parent palm, child palm_collision_ball_6, origin xyz=0.02 0.0 0.026  rpy=0 0 0
- added joint palm_collision_ball_7_joint: type fixed, parent palm, child palm_collision_ball_7, origin xyz=-0.02 0.0 0.026  rpy=0 0 0
- added joint palm_collision_ball_8_joint: type fixed, parent palm, child palm_collision_ball_8, origin xyz=-0.02 0.0 0.05 rpy=0 0 0
- added joint palm_collision_ball_9_joint: type fixed, parent palm, child palm_collision_ball_9, origin xyz=-0.02 0.0 0.076 rpy=0 0 0
