Commit message: update

File: robots/hands/allegro_hand/allegro_hand_right_dummy_ball.urdf (robot description, URDF)
Before this commit: robot allegro_right, 39 links, 38 joints
Links:
- removed link link_0.0_fsr
- removed link link_1.0_fsr
- removed link link_10.0_fsr
- removed link link_11.0_tip_fsr
- removed link link_14.0_fsr
- removed link link_15.0_fsr
- removed link link_15.0_tip_fsr
- removed link link_2.0_fsr
- removed link link_3.0_tip_fsr
- removed link link_4.0_fsr
- removed link link_5.0_fsr
- removed link link_6.0_fsr
- removed link link_7.0_tip_fsr
- removed link link_8.0_fsr
- removed link link_9.0_fsr
- removed link link_base_fsr
- added link base_link_pitch
- added link base_link_roll
- added link base_link_x
- added link base_link_y
- added link base_link_yaw
- added link base_link_z
- link base_link: geometry collision box size=0.0414 0.0538 0.0428; collision box size=0.0414 0.0720 0.013
- link link_0.0: geometry collision box size=0.0196 0.0275 0.0164; visual mesh filename=meshes/visual/link_0.0.obj
- link link_1.0: geometry collision box size=0.0196 0.0275 0.054; visual mesh filename=meshes/visual/link_1.0.obj
- link link_10.0: geometry collision box size=0.0196 0.0275 0.0384; visual mesh filename=meshes/visual/link_2.0.obj
- link link_11.0: geometry collision box size=0.0196 0.0269 0.022; visual mesh filename=meshes/visual/link_3.0.obj
- link link_11.0_tip: mass None -> 0.0168; geometry collision mesh filename=meshes/collision/link_tip.obj; visual mesh filename=meshes/visual/link_tip.obj
- link link_12.0: geometry collision box size=0.0358 0.034 0.0455; visual mesh filename=meshes/visual/link_12.0_right.obj
- link link_13.0: geometry collision box size=0.0196 0.0275 0.0177; visual mesh filename=meshes/visual/link_13.0.obj
- link link_14.0: geometry collision box size=0.0196 0.0275 0.0514; visual mesh filename=meshes/visual/link_14.0.obj
- link link_15.0: geometry collision box size=0.0196 0.0269 0.04; visual mesh filename=meshes/visual/link_15.0.obj
- link link_15.0_tip: mass None -> 0.0168; geometry collision mesh filename=meshes/collision/link_tip.obj; visual mesh filename=meshes/visual/link_tip.obj
- link link_2.0: geometry collision box size=0.0196 0.0275 0.0384; visual mesh filename=meshes/visual/link_2.0.obj
- link link_3.0: geometry collision box size=0.0196 0.0269 0.022; visual mesh filename=meshes/visual/link_3.0.obj
- link link_3.0_tip: mass None -> 0.0168; geometry collision mesh filename=meshes/collision/link_tip.obj; visual mesh filename=meshes/visual/link_tip.obj
- link link_4.0: geometry collision box size=0.0196 0.0275 0.0164; visual mesh filename=meshes/visual/link_0.0.obj
- link link_5.0: geometry collision box size=0.0196 0.0275 0.054; visual mesh filename=meshes/visual/link_1.0.obj
- link link_6.0: geometry collision box size=0.0196 0.0275 0.0384; visual mesh filename=meshes/visual/link_2.0.obj
- link link_7.0: geometry collision box size=0.0196 0.0269 0.022; visual mesh filename=meshes/visual/link_3.0.obj
- link link_7.0_tip: mass None -> 0.0096; geometry collision mesh filename=meshes/collision/link_tip.obj; visual mesh filename=meshes/visual/link_tip.obj
- link link_8.0: geometry collision box size=0.0196 0.0275 0.0164; visual mesh filename=meshes/visual/link_0.0.obj
- link link_9.0: geometry collision box size=0.0196 0.0275 0.054; visual mesh filename=meshes/visual/link_1.0.obj
Joints:
- removed joint joint_0.0_fsr
- removed joint joint_1.0_fsr
- removed joint joint_10.0_fsr
- removed joint joint_11.0_tip_fsr
- removed joint joint_14.0_fsr
- removed joint joint_15.0_fsr
- removed joint joint_15.0_tip_fsr
- removed joint joint_2.0_fsr
- removed joint joint_3.0_tip_fsr
- removed joint joint_4.0_fsr
- removed joint joint_5.0_fsr
- removed joint joint_6.0_fsr
- removed joint joint_7.0_tip_fsr
- removed joint joint_8.0_fsr
- removed joint joint_9.0_fsr
- removed joint joint_base_fsr
- added joint dummy_x_rotation_joint: type revolute, parent base_link_roll, child base_link_pitch, origin xyz=0 0 0 rpy=0 0 0, axis 1 0 0, limit lower=-6.283185 upper=6.283185 effort=100.95 velocity=108.48
- added joint dummy_x_translation_joint: type prismatic, parent base_link_x, child base_link_y, origin xyz=0 0 0 rpy=0 0 0, axis 1 0 0, limit lower=-10 upper=10 effort=300 velocity=2.1750
- added joint dummy_y_rotation_joint: type revolute, parent base_link_pitch, child base_link_yaw, origin xyz=0 0 0 rpy=0 0 0, axis 0 1 0, limit lower=-6.283185 upper=6.283185 effort=100.95 velocity=108.48
- added joint dummy_y_translation_joint: type prismatic, parent base_link_y, child base_link_z, origin xyz=0 0 0 rpy=0 0 0, axis 0 1 0, limit lower=-10 upper=10 effort=300 velocity=2.1750
- added joint dummy_z_rotation_joint: type revolute, parent base_link_yaw, child base_link, origin xyz=0 0 0 rpy=0 0 0, axis 0 0 1, limit lower=-6.283185 upper=6.283185 effort=100.95 velocity=108.48
- added joint dummy_z_translation_joint: type prismatic, parent base_link_z, child base_link_roll, origin xyz=0 0 0 rpy=0 0 0, axis 0 0 1, limit lower=-10 upper=10 effort=300 velocity=2.1750
